File: engineering/Night_light_timer.sch (EAGLE design)
At the start: 11 parts, among them IC2 LP2951D, Q1 FDN360P, Y1 16MHz

Commit message: initial work
Parts:
- removed C1, C2: (no value), capacitor-wima:C2,5-3
- removed D1: Yellow, SparkFun-LED:LED-YELLOW0603
- removed IC1, IC3: (no value), linear:2CMPD
- removed IC2: LP2951D, linear:LP2951D
- removed Q1: FDN360P, transistor-power:FDN360P
- removed R1, R4: (no value), rcl:R-US_0204/5
- removed R3: (no value), resistor:R-US_0204/7
- removed Y1: 16MHz, SparkFun-Clocks:RESONATOR-16MHZSMD_3.2X1.3
Connections:
- removed net +5V: C1.1, IC2.IN, IC2.SH-DOWN, Q1.D, Q1.S
- removed net GND: C1.2, C2.2, D1.C, IC2.!ERROR, R4.1
- removed net N$1: R3.2
- removed net N$2: IC1.OUT, Q1.G
- removed net N$3: IC1.+IN, R3.1, R4.2
- removed net N$4: IC3.+IN
- removed net N$5: C2.1, IC2.OUT
- removed net N$6: IC3.OUT
- removed net N$7: IC3.-IN, R1.2
- removed net N$8: D1.A, R1.1
Changed lines of the file:
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@@
 <parts>
 <part name="FRAME1" library="frames" deviceset="DINA4_L" device=""/>
-<part name="Y1" library="SparkFun-Clocks" deviceset="RESONATOR-16MHZ" device="SMD_3.2X1.3" value="16MHz"/>
-<part name="C1" library="capacitor-wima" deviceset="C" device="2,5-3"/>
-<part name="P+2" library="supply1" deviceset="+5V" device=""/>
-<part name="GND2" library="SparkFun-PowerSymbols" deviceset="GND" device=""/>
-<part name="R3" library="resistor" deviceset="R-US_" device="0204/7"/>
-<part name="R4" library="rcl" deviceset="R-US_" device="0204/5"/>
-<part name="GND3" library="SparkFun-PowerSymbols" deviceset="GND" device=""/>
-<part name="IC1" library="linear" deviceset="2CMP" device="D"/>
-<part name="Q1" library="transistor-power" deviceset="FDN360P" device=""/>
-<part name="P+3" library="supply1" deviceset="+5V" device=""/>
-<part name="IC2" library="linear" deviceset="LP2951" device="D"/>
-<part name="GND1" library="SparkFun-PowerSymbols" deviceset="GND" device=""/>
-<part name="C2" library="capacitor-wima" deviceset="C" device="2,5-3"/>
-<part name="GND4" library="SparkFun-PowerSymbols" deviceset="GND" device=""/>
-<part name="IC3" library="linear" deviceset="2CMP" device="D"/>
-<part name="R1" library="rcl" deviceset="R-US_" device="0204/5"/>
-<part name="D1" library="SparkFun-LED" deviceset="LED-YELLOW" device="0603" value="Yellow"/>
-<part name="GND5" library="SparkFun-PowerSymbols" deviceset="GND" device=""/>
 </parts>
 <sheets>
@@
 <instance part="FRAME1" gate="G$1" x="0" y="0"/>
 <instance part="FRAME1" gate="G$2" x="162.56" y="0"/>
-<instance part="Y1" gate="G$1" x="55.88" y="109.22"/>
-<instance part="C1" gate="G$1" x="15.24" y="167.64"/>
-<instance part="P+2" gate="1" x="10.16" y="175.26"/>
-<instance part="GND2" gate="1" x="10.16" y="157.48"/>
-<instance part="R3" gate="G$1" x="40.64" y="165.1" rot="R90"/>
-<instance part="R4" gate="G$1" x="40.64" y="152.4" rot="R90"/>
-<instance part="GND3" gate="1" x="40.64" y="142.24"/>
-<instance part="IC1" gate="A" x="68.58" y="154.94"/>
-<instance part="Q1" gate="G$1" x="71.12" y="127" rot="R270"/>
-<instance part="P+3" gate="1" x="86.36" y="127"/>
-<instance part="IC2" gate="G$1" x="114.3" y="116.84"/>
-<instance part="GND1" gate="1" x="93.98" y="104.14"/>
-<instance part="C2" gate="G$1" x="132.08" y="119.38"/>
-<instance part="GND4" gate="1" x="132.08" y="109.22"/>
-<instance part="IC3" gate="A" x="116.84" y="147.32"/>
-<instance part="R1" gate="G$1" x="132.08" y="149.86" rot="R90"/>
-<instance part="D1" gate="G$1" x="132.08" y="139.7"/>
-<instance part="GND5" gate="1" x="132.08" y="129.54"/>
 </instances>
 <busses>
 </busses>
 <nets>
-<net name="GND" class="0">
-<segment>
-<pinref part="C1" gate="G$1" pin="2"/>
-<wire x1="15.24" y1="162.56" x2="15.24" y2="160.02" width="0.1524" layer="91"/>
-<wire x1="15.24" y1="160.02" x2="10.16" y2="160.02" width="0.1524" layer="91"/>
-<wire x1="10.16" y1="160.02" x2="5.08" y2="160.02" width="0.1524" layer="91"/>
-<wire x1="5.08" y1="160.02" x2="5.08" y2="165.1" width="0.1524" layer="91"/>
-<pinref part="GND2" gate="1" pin="GND"/>
-<junction x="10.16" y="160.02"/>
-</segment>
-<segment>
-<pinref part="R4" gate="G$1" pin="1"/>
-<pinref part="GND3" gate="1" pin="GND"/>
-<wire x1="40.64" y1="147.32" x2="40.64" y2="144.78" width="0.1524" layer="91"/>
-</segment>
-<segment>
-<pinref part="IC2" gate="G$1" pin="!ERROR"/>
-<wire x1="101.6" y1="109.22" x2="93.98" y2="109.22" width="0.1524" layer="91"/>
-<pinref part="GND1" gate="1" pin="GND"/>
-<wire x1="93.98" y1="109.22" x2="93.98" y2="106.68" width="0.1524" layer="91"/>
-</segment>
-<segment>
-<pinref part="C2" gate="G$1" pin="2"/>
-<pinref part="GND4" gate="1" pin="GND"/>
-<wire x1="132.08" y1="114.3" x2="132.08" y2="111.76" width="0.1524" layer="91"/>
-</segment>
-<segment>
-<pinref part="D1" gate="G$1" pin="C"/>
-<pinref part="GND5" gate="1" pin="GND"/>
-<wire x1="132.08" y1="134.62" x2="132.08" y2="132.08" width="0.1524" layer="91"/>
-</segment>
-</net>
-<net name="+5V" class="0">
-<segment>
-<pinref part="C1" gate="G$1" pin="1"/>
-<wire x1="15.24" y1="170.18" x2="15.24" y2="172.72" width="0.1524" layer="91"/>
-<wire x1="15.24" y1="172.72" x2="10.16" y2="172.72" width="0.1524" layer="91"/>
-<wire x1="10.16" y1="172.72" x2="5.08" y2="172.72" width="0.1524" layer="91"/>
-<wire x1="5.08" y1="172.72" x2="5.08" y2="167.64" width="0.1524" layer="91"/>
-<pinref part="P+2" gate="1" pin="+5V"/>
-<junction x="10.16" y="172.72"/>
-</segment>
-<segment>
-<pinref part="Q1" gate="G$1" pin="D"/>
-<wire x1="66.04" y1="124.46" x2="53.34" y2="124.46" width="0.1524" layer="91"/>
-<pinref part="Q1" gate="G$1" pin="S"/>
-<wire x1="66.04" y1="124.46" x2="76.2" y2="124.46" width="0.1524" layer="91"/>
-<wire x1="76.2" y1="124.46" x2="86.36" y2="124.46" width="0.1524" layer="91"/>
-<junction x="76.2" y="124.46"/>
-<pinref part="P+3" gate="1" pin="+5V"/>
-<wire x1="86.36" y1="124.46" x2="93.98" y2="124.46" width="0.1524" layer="91"/>
-<junction x="86.36" y="124.46"/>
-<wire x1="93.98" y1="116.84" x2="93.98" y2="124.46" width="0.1524" layer="91"/>
-<wire x1="93.98" y1="124.46" x2="101.6" y2="124.46" width="0.1524" layer="91"/>
-<junction x="93.98" y="124.46"/>
-<pinref part="IC2" gate="G$1" pin="IN"/>
-<pinref part="IC2" gate="G$1" pin="SH-DOWN"/>
-<wire x1="93.98" y1="116.84" x2="101.6" y2="116.84" width="0.1524" layer="91"/>
-</segment>
-</net>
-<net name="N$3" class="0">
-<segment>
-<pinref part="R3" gate="G$1" pin="1"/>
-<pinref part="R4" gate="G$1" pin="2"/>
-<wire x1="40.64" y1="160.02" x2="40.64" y2="157.48" width="0.1524" layer="91"/>
-<wire x1="40.64" y1="160.02" x2="58.42" y2="160.02" width="0.1524" layer="91"/>
-<junction x="40.64" y="160.02"/>
-<wire x1="58.42" y1="160.02" x2="58.42" y2="157.48" width="0.1524" layer="91"/>
-<wire x1="58.42" y1="157.48" x2="60.96" y2="157.48" width="0.1524" layer="91"/>
-<pinref part="IC1" gate="A" pin="+IN"/>
-</segment>
-</net>
-<net name="N$1" class="0">
-<segment>
-<pinref part="R3" gate="G$1" pin="2"/>
-<wire x1="40.64" y1="170.18" x2="40.64" y2="177.8" width="0.1524" layer="91"/>
-<wire x1="40.64" y1="177.8" x2="27.94" y2="177.8" width="0.1524" layer="91"/>
-</segment>
-</net>
-<net name="N$2" class="0">
-<segment>
-<pinref part="IC1" gate="A" pin="OUT"/>
-<wire x1="76.2" y1="154.94" x2="86.36" y2="154.94" width="0.1524" layer="91"/>
-<wire x1="86.36" y1="154.94" x2="86.36" y2="137.16" width="0.1524" layer="91"/>
-<wire x1="86.36" y1="137.16" x2="73.66" y2="137.16" width="0.1524" layer="91"/>
-<wire x1="73.66" y1="137.16" x2="73.66" y2="129.54" width="0.1524" layer="91"/>
-<pinref part="Q1" gate="G$1" pin="G"/>
-</segment>
-</net>
-<net name="N$5" class="0">
-<segment>
-<pinref part="IC2" gate="G$1" pin="OUT"/>
-<wire x1="127" y1="124.46" x2="132.08" y2="124.46" width="0.1524" layer="91"/>
-<wire x1="132.08" y1="124.46" x2="132.08" y2="121.92" width="0.1524" layer="91"/>
-<pinref part="C2" gate="G$1" pin="1"/>
-</segment>
-</net>
-<net name="N$4" class="0">
-<segment>
-<pinref part="IC3" gate="A" pin="+IN"/>
-<wire x1="109.22" y1="149.86" x2="99.06" y2="149.86" width="0.1524" layer="91"/>
-</segment>
-</net>
-<net name="N$7" class="0">
-<segment>
-<pinref part="IC3" gate="A" pin="-IN"/>
-<wire x1="109.22" y1="144.78" x2="109.22" y2="137.16" width="0.1524" layer="91"/>
-<wire x1="109.22" y1="137.16" x2="127" y2="137.16" width="0.1524" layer="91"/>
-<wire x1="127" y1="137.16" x2="127" y2="157.48" width="0.1524" layer="91"/>
-<wire x1="127" y1="157.48" x2="132.08" y2="157.48" width="0.1524" layer="91"/>
-<pinref part="R1" gate="G$1" pin="2"/>
-<wire x1="132.08" y1="157.48" x2="132.08" y2="154.94" width="0.1524" layer="91"/>
-</segment>
-</net>
-<net name="N$6" class="0">
-<segment>
-<pinref part="IC3" gate="A" pin="OUT"/>
-<wire x1="124.46" y1="147.32" x2="127" y2="147.32" width="0.1524" layer="91"/>
-</segment>
-</net>
-<net name="N$8" class="0">
-<segment>
-<pinref part="R1" gate="G$1" pin="1"/>
-<pinref part="D1" gate="G$1" pin="A"/>
-<wire x1="132.08" y1="144.78" x2="132.08" y2="142.24" width="0.1524" layer="91"/>
-</segment>
-</net>
 </nets>
 </sheet>
